File: Schematic/Mainboard/zx2022.kicad_pcb (KiCad board)
At the start: 2 copper layers, 100 x 100 mm, 34 parts, among them J2 Bus, J3 Terminal, J4 Ser. Disk, J5 PATA, J6 Power, J7 PS/2 Keyoard, SW1 Reset, U1 Z80CPU, U2 628128, U3 28C256_PLC32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

Commit message: Board version 1.2
Parts:
- moved J7 0.07 mm to (237.5, 66.3)
Connections:
- J7 pad 1: +5V -> GND
- J7 pad 2: /~{RIA} -> /~{RIB}
- J7 pad 3: /~{RIB} -> /~{RIA}
- J7 pad 4: GND -> +5V
Routing:
- net /~{RIB}: track 210.7 -> 214.2 mm, vias 1 -> 2
- net +5V: track 484.3 -> 486.4 mm
Other:
- board text added: "ZX2022 Rev 1.2"
- board text removed: "ZX2022 Rev 1.1"
