File: Schematic/Mainboard/zx2022.kicad_sch (KiCad schematic)
At the start: 35 parts, among them J2 Bus, J3 Terminal, J4 Ser. Disk, J5 PATA, J6 Power, J7 PS/2 Keyoard, SW1 Reset, U2 628128, U3 28C256_PLC32, U4 Z80DART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

Commit message: Board version 1.2
Parts:
- U1: value (none) -> Z80CPU; footprint (none) -> Package_DIP:DIP-40_W15.24mm_Socket
Connections:
- net +5V: now also J7.4 (Pin_4); no longer J7.1 (Pin_1)
- net GND: now also J7.1 (Pin_1); no longer J7.4 (Pin_4)
- net ~{RIA}: now also J7.3 (Pin_3); no longer J7.2 (Pin_2)
- net ~{RIB}: now also J7.2 (Pin_2); no longer J7.3 (Pin_3)
Other:
- moved on the sheet: J7
Changed lines of the file:
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@@
       (effects (font (size 1.27 1.27)) (justify left))
     )
-    (property "Value" "" (id 1) (at 91.44 69.85 0)
-      (effects (font (size 1.27 1.27)) (justify left))
-    )
-    (property "Footprint" "" (id 2) (at 96.52 68.58 0)
+    (property "Value" "Z80CPU" (id 1) (at 91.44 69.85 0)
+      (effects (font (size 1.27 1.27)) (justify left))
+    )
+    (property "Footprint" "Package_DIP:DIP-40_W15.24mm_Socket" (id 2) (at 96.52 68.58 0)
       (effects (font (size 1.27 1.27)) hide)
     )
@@
     (pin "1")
   )
-  (symbol (lib_id "Connector:Conn_01x04_Male") (at 337.185 223.52 0) (mirror y) (unit 1)
-    (in_bom yes) (on_board yes)
-    (property "Reference" "J7" (id 0) (at 336.55 215.9 0))
-    (property "Value" "PS/2 Keyoard" (id 1) (at 340.995 232.41 0))
-    (property "Footprint" "zx2022:PinHeader_1x04_P2.54mm_Horizontal" (id 2) (at 337.185 223.52 0)
-      (effects (font (size 1.27 1.27)) hide)
-    )
-    (property "Datasheet" "~" (id 3) (at 337.185 223.52 0)
-      (effects (font (size 1.27 1.27)) hide)
-    )
+  (symbol (lib_id "Connector:Conn_01x04_Male") (at 337.185 226.06 180) (unit 1)
+    (in_bom yes) (on_board yes)
+    (property "Reference" "J7" (id 0) (at 336.55 233.68 0))
+    (property "Value" "PS/2 Keyoard" (id 1) (at 340.995 217.17 0))
+    (property "Footprint" "zx2022:PinHeader_1x04_P2.54mm_Horizontal" (id 2) (at 337.185 226.06 0)
+      (effects (font (size 1.27 1.27)) hide)
+    )
+    (property "Datasheet" "~" (id 3) (at 337.185 226.06 0)
+      (effects (font (size 1.27 1.27)) hide)
+    )
